File: PowerIO.kicad_sch (KiCad schematic)
At the start: 14 parts, among them Q7 BTN8982TA

Commit message: Added ethernet and ntcs
Parts:
- removed D1: 3v, Diode_SMD:D_SOD-123, symbol Device:D_Zener
- removed R41: 1k, Resistor_SMD:R_0805_2012Metric, symbol Device:R
- added C15: 1.5nF, Capacitor_SMD:C_0603_1608Metric, symbol Device:C
- R25: value 3k -> 3.3k
- R57: value 5.1k -> 0R; footprint Resistor_SMD:R_0805_2012Metric -> Resistor_SMD:R_0805_2012Metric_Pad1.20x1.40mm_HandSolder
- R8: value 6k -> 33k
Connections:
- net GND: now also C15.2
- net IN: now also R25.1, R8.2, C15.1
Other:
- moved on the sheet: C6, R10, R11, R25, R8
