File: MildlyOverkill.kicad_sch (KiCad schematic)
At the start: 104 parts, among them J1 USB_C_Receptacle_USB2.0_16P, J2 Screw_Terminal_01x02, J3 Motors, J4 IO, J5 Conn_01x04_Pin, J6 Conn_01x04_MountingPin, J8 RJ45_Wuerth_7499010211A, J9 Analog, M1 Fan_4pin, Q1 Q_PMOS_GDS, U1 ESP32-S3-WROOM-1, U2 MCP3208, U3 LD1117S33TR_SOT223, U5 USBLC6-2P6, U6 TPS62932, U7 W5500, Y1 3134250001

Commit message: idk where to begin...
Parts:
- removed C21, C36, C37, C38, C39, C40, C41: 0.1uF, Capacitor_SMD:C_0603_1608Metric, symbol Device:C
- removed C26, C35: 10uF 16V, Capacitor_THT:CP_Radial_D4.0mm_P2.00mm, symbol Device:C_Polarized
- removed C27: 4.7uF, Capacitor_SMD:C_1206_3216Metric, symbol Device:C
- removed C28: 10nF, Capacitor_SMD:C_0805_2012Metric, symbol Device:C
- removed C29, C30, C31: 10nF, Capacitor_SMD:C_0603_1608Metric, symbol Device:C
- removed C32: 22nF, Capacitor_SMD:C_0603_1608Metric, symbol Device:C
- removed C33, C34: 18pF, Capacitor_SMD:C_0805_2012Metric, symbol Device:C
- removed C42: 1nF 10kV, Capacitor_SMD:C_1206_3216Metric, symbol Device:C
- removed FB2: GZ2012D121TF, Inductor_SMD:L_0805_2012Metric, symbol Device:FerriteBead
- removed J8: RJ45_Wuerth_7499010211A, Connector_RJ:RJ45_Wuerth_7499010211A_Horizontal, symbol Connector:RJ45_Wuerth_7499010211A
- removed R41: 12.4K, Resistor_SMD:R_0805_2012Metric, symbol Device:R
- removed R42, R43: 82, Resistor_SMD:R_0603_1608Metric, symbol Device:R
- removed R44, R62: 49, Resistor_SMD:R_0603_1608Metric, symbol Device:R
- removed R64, R65, R67, R68: 33, Resistor_SMD:R_0603_1608Metric, symbol Device:R
- removed R66: 10, Resistor_SMD:R_0603_1608Metric, symbol Device:R
- removed R73: 1M, Resistor_SMD:R_0805_2012Metric, symbol Device:R
- removed R74: 0, Resistor_SMD:R_0805_2012Metric_Pad1.20x1.40mm_HandSolder, symbol Device:R
- removed R75, R76: 330, Resistor_SMD:R_0805_2012Metric, symbol Device:R
- removed U7: W5500, Package_QFP:LQFP-48_7x7mm_P0.5mm, symbol Interface_Ethernet:W5500
- removed Y1: 3134250001, Crystal:Crystal_SMD_3225-4Pin_3.2x2.5mm, symbol Device:Crystal_GND24
- added J7: GND, TerminalBlock_Phoenix:TerminalBlock_Phoenix_MPT-0,5-4-2.54_1x04_P2.54mm_Horizontal, symbol Connector:Screw_Terminal_01x04
- added J8: VCC, TerminalBlock_Phoenix:TerminalBlock_Phoenix_MPT-0,5-4-2.54_1x04_P2.54mm_Horizontal, symbol Connector:Screw_Terminal_01x04
- R1, R12, R13, R14, R15, R16, R17, R18, R19, R3, R4, R5, R52, R53, R54, R55, R56, R57, R61, R77: footprint Resistor_SMD:R_0805_2012Metric -> Resistor_SMD:R_0603_1608Metric
Connections:
- net GND: now also J7.1 (Pin_1), J7.2 (Pin_2), J7.3 (Pin_3), J7.4 (Pin_4)
- net VCC: now also J8.1 (Pin_1), J8.2 (Pin_2), J8.3 (Pin_3), J8.4 (Pin_4)
- no-connect marks 25 -> 12
Other:
- moved on the sheet: D5, FB1, H1, H2, H3, H4, J1, J6, R3, R5, U5

Commit message: I cant do this anymore
Signed-off-by: Peter Schmidt <hackepetersilie@gmx.de>
Parts:
- added J10: Conn_01x07_Pin, Connector_PinSocket_2.54mm:PinSocket_1x07_P2.54mm_Vertical, symbol Connector:Conn_01x07_Pin
- added J11: Conn_01x08_Pin, Connector_PinSocket_2.54mm:PinSocket_1x08_P2.54mm_Vertical, symbol Connector:Conn_01x08_Pin
Connections:
- net +3.3V: now also J11.2 (Pin_2)
- net +5V: now also J11.1 (Pin_1)
- net GND: now also J10.7 (Pin_7), J11.3 (Pin_3), J11.8 (Pin_8)
- net MISO: now also J11.5 (Pin_5)
- net MOSI: now also J11.6 (Pin_6)
- net SCLK: now also J11.4 (Pin_4)
- net Pin1: now reaches U1.19 (IO11)
- net Pin1: now also J10.1 (Pin_1)
- net Pin2: now reaches U1.20 (IO12)
- net Pin2: now also J10.2 (Pin_2)
- net Pin3: now reaches U1.21 (IO13)
- net Pin3: now also J10.3 (Pin_3)
- net Pin4: now reaches U1.22 (IO14)
- net Pin4: now also J10.4 (Pin_4)
- net Pin5: now reaches U1.24 (IO47)
- net Pin5: now also J10.5 (Pin_5)
- net Pin6: now reaches U1.25 (IO48)
- net Pin6: now also J10.6 (Pin_6)
- net ETH_CS renamed Pin7
- net Pin7: now also J11.7 (Pin_7)
- no-connect marks 12 -> 6
