File: MildlyOverkill.kicad_sch (KiCad schematic)
At the start: 73 parts, among them J1 USB_C_Receptacle_USB2.0_16P, J10 Conn_01x07_Pin, J11 Conn_01x08_Pin, J2 Screw_Terminal_01x02, J3 Motors, J4 IO, J5 Conn_01x04_Pin, J6 Conn_01x04_MountingPin, J7 GND, J8 VCC, J9 Analog, Q1 AOD4185, U1 ESP32-S3-WROOM-1, U2 MCP3208, U3 LD1117S33TR_SOT223, U5 USBLC6-2P6, U6 TPS62932

Commit message: BOM cleanup: values, MPNs and voltage ratings from todo.md
Values/fields only, no footprint or net changes (netlist diff is empty).

Co-Authored-By: Claude Sonnet 5.5 <noreply@anthropic.com> (obviously)
Parts:
- C1: value 100nF -> 1uF 10V
- C11: value 47uF -> 47uF 10V X5R
- C13: value 100nF -> 100nF 50V
- C14: value 10uF -> 10uF 50V
- C16: value 1000uF -> 1000uF 35V
- C17: value 10uF -> 10uF 10V X5R
- C20: value 22uF -> 22uF 10V X5R
- D4: value SMAJ33A -> SMAJ24CA
- F1: value Fuse -> 10A
- R1: value 5,1K -> 10k
- R3, R5: value 5,1K -> 5.1k
- R54: value 400 -> 402
- R77: value R -> 10k 1%
- TH1: value Thermistor_NTC -> NCP18XH103F03RB
- U3: value LD1117S33TR_SOT223 -> AP7361C-33ER-13
Changed lines of the file:
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@@
 			)
 		)
-		(property "Value" "R"
+		(property "Value" "10k 1%"
 			(at 262.89 93.9799 0)
 			(show_name no)
@@
 			)
 		)
-		(property "Value" "LD1117S33TR_SOT223"
+		(property "Value" "AP7361C-33ER-13"
 			(at 218.44 39.37 0)
 			(show_name no)
@@
 			)
 		)
-		(property "Value" "SMAJ33A"
+		(property "Value" "SMAJ24CA"
 			(at 40.64 43.1799 90)
 			(show_name no)
@@
 			)
 		)
-		(property "Value" "Fuse"
+		(property "Value" "10A"
 			(at 33.02 34.29 90)
 			(show_name no)
@@
 			)
 		)
-		(property "Value" "100nF"
+		(property "Value" "1uF 10V"
 			(at 219.71 102.8699 0)
 			(show_name no)
@@
 			)
 		)
-		(property "Value" "22uF"
+		(property "Value" "22uF 10V X5R"
 			(at 275.59 135.8899 0)
 			(show_name no)
@@
 			)
 		)
-		(property "Value" "1000uF"
+		(property "Value" "1000uF 35V"
 			(at 80.01 42.2909 0)
 			(show_name no)
@@
 			)
 		)
-		(property "Value" "100nF"
+		(property "Value" "100nF 50V"
 			(at 110.49 45.7199 0)
 			(show_name no)
@@
 			)
 		)
-		(property "Value" "5,1K"
+		(property "Value" "5.1k"
 			(at 351.79 55.118 90)
 			(show_name no)
@@
 			)
 		)
-		(property "Value" "10uF"
+		(property "Value" "10uF 10V X5R"
 			(at 175.26 34.2899 0)
 			(show_name no)
@@
 			)
 		)
-		(property "Value" "10uF"
+		(property "Value" "10uF 50V"
 			(at 97.79 50.7999 0)
 			(show_name no)
@@
 			)
 		)
-		(property "Value" "Thermistor_NTC"
+		(property "Value" "NCP18XH103F03RB"
 			(at 262.89 103.1874 0)
 			(hide yes)
@@
 			)
 		)
-		(property "Value" "5,1K"
+		(property "Value" "10k"
 			(at 218.44 91.4399 0)
 			(show_name no)
@@
 			)
 		)
-		(property "Value" "5,1K"
+		(property "Value" "5.1k"
 			(at 351.79 46.736 90)
 			(show_name no)
@@
 			)
 		)
-		(property "Value" "400"
+		(property "Value" "402"
 			(at 184.15 95.2499 0)
 			(show_name no)
@@
 			)
 		)
-		(property "Value" "47uF"
+		(property "Value" "47uF 10V X5R"
 			(at 160.02 52.0699 0)
 			(show_name no)
