File: MildlyOverkill.kicad_sch (KiCad schematic)
At the start: 73 parts, among them J1 USB_C_Receptacle_USB2.0_16P, J10 Conn_01x07_Pin, J11 Conn_01x08_Pin, J2 Screw_Terminal_01x02, J3 Motors, J4 IO, J5 Conn_01x04_Pin, J6 Conn_01x04_MountingPin, J7 GND, J8 VCC, J9 Analog, Q1 AOD4185, U1 ESP32-S3-WROOM-1, U2 MCP3208, U3 AP7361C-33ER-13, U5 USBLC6-2P6, U6 TPS62932

Commit message: Did some stuff on the todo list TL;DR:The piece of meat did what the thinking sand said and now it can sleep in peace. The end.
Parts:
- removed U3: AP7361C-33ER-13, Package_TO_SOT_SMD:SOT-223-3_TabPin2, symbol Regulator_Linear:LD1117S33TR_SOT223
- added C25: 2.2uF, Capacitor_SMD:C_1206_3216Metric, symbol Device:C
- added R20, R21: 4.7k, Resistor_SMD:R_0805_2012Metric_Pad1.20x1.40mm_HandSolder, symbol Device:R
- added U3: AP7361C-33E, Package_TO_SOT_SMD:SOT-223-3_TabPin2, symbol Regulator_Linear:AP7361C-33E
- D3: footprint Diode_SMD:D_0805_2012Metric -> Diode_SMD:D_SOD-123
- D5: footprint Diode_SMD:D_SOD-323 -> Diode_SMD:D_SOD-123
Connections:
- net +3.3V: now also R20.2, R21.2, U3.3 (VO)
- net +5V: now also U3.1 (VI)
- net GND: now also C25.2, U3.2 (GND)
- net SCL: now also R20.1
- net SDA: now also R21.1
- net at D5.2 (A), FB1.2: now also C25.1
Other:
- moved on the sheet: D5, FB1
