File: MildlyOverkill.kicad_pcb (KiCad board)
At the start: 4 copper layers, 100 x 80 mm, 139 parts, among them J1 USB_C_Receptacle_USB2.0_16P, J2 Screw_Terminal_01x02, J3 Motors, J4 IO, J5 Conn_01x04_Pin, J6 Conn_01x04_MountingPin, J8 RJ45_Wuerth_7499010211A, J9 Analog, M1 Fan_4pin, Q1 Q_PMOS_GDS, U1 ESP32-S3-WROOM-1, U2 MCP3208, U3 LD1117S33TR_SOT223, U4 TPS4H160AQPWPRQ1, U5 USBLC6-2P6, U6 TPS62932, U7 W5500, U8 DRV8874PWPR, U9 DRV8874PWPR, Y1 3134250001

Commit message: idk where to begin...
Parts:
- removed C21, C36, C37, C38, C39, C40, C41: 0.1uF, Capacitor_SMD:C_0603_1608Metric
- removed C26, C35: 10uF 16V, Capacitor_THT:CP_Radial_D4.0mm_P2.00mm
- removed C27: 4.7uF, Capacitor_SMD:C_1206_3216Metric
- removed C28: 10nF, Capacitor_SMD:C_0805_2012Metric
- removed C29, C30, C31: 10nF, Capacitor_SMD:C_0603_1608Metric
- removed C32: 22nF, Capacitor_SMD:C_0603_1608Metric
- removed C33, C34: 18pF, Capacitor_SMD:C_0805_2012Metric
- removed C42: 1nF 10kV, Capacitor_SMD:C_1206_3216Metric
- removed FB2: GZ2012D121TF, Inductor_SMD:L_0805_2012Metric
- removed R41: 12.4K, Resistor_SMD:R_0805_2012Metric
- removed R42, R43: 82, Resistor_SMD:R_0603_1608Metric
- removed R44, R62: 49, Resistor_SMD:R_0603_1608Metric
- removed R64, R65, R67, R68: 33, Resistor_SMD:R_0603_1608Metric
- removed R66: 10, Resistor_SMD:R_0603_1608Metric
- removed R73: 1M, Resistor_SMD:R_0805_2012Metric
- removed R74: 0, Resistor_SMD:R_0805_2012Metric_Pad1.20x1.40mm_HandSolder
- removed R75, R76: 330, Resistor_SMD:R_0805_2012Metric
- removed U7: W5500, Package_QFP:LQFP-48_7x7mm_P0.5mm
- removed Y1: 3134250001, Crystal:Crystal_SMD_3225-4Pin_3.2x2.5mm
- removed kibuzzard-6AB94CCA: G***, kibuzzard-6AB94CCA
- removed kibuzzard-6AB94CD2: G***, kibuzzard-6AB94CD2
- removed kibuzzard-6AB94CD7: G***, kibuzzard-6AB94CD7
- removed kibuzzard-6AB94CDC: G***, kibuzzard-6AB94CDC
- removed kibuzzard-6AB94D65: G***, kibuzzard-6AB94D65
- removed kibuzzard-6AB94D6B: G***, kibuzzard-6AB94D6B
- removed kibuzzard-6AB94D6F: G***, kibuzzard-6AB94D6F
- removed kibuzzard-6AB94D73: G***, kibuzzard-6AB94D73
- added D11: LED, LED_SMD:LED_0603_1608Metric, F.Cu at (125.0, 42.0)
- added D12: LED, LED_SMD:LED_0603_1608Metric, F.Cu at (122.0, 42.0)
- added D13: LED, LED_SMD:LED_0603_1608Metric, F.Cu at (119.0, 42.0)
- added D23: LED, LED_SMD:LED_0603_1608Metric, F.Cu at (116.0, 42.0)
- added J10: Conn_01x07_Pin, Connector_PinSocket_2.54mm:PinSocket_1x07_P2.54mm_Vertical, F.Cu at (97.5, 54.8)
- added J11: Conn_01x08_Pin, Connector_PinSocket_2.54mm:PinSocket_1x08_P2.54mm_Vertical, F.Cu at (172.5, 55.0)
- added J7: GND, TerminalBlock_Phoenix:TerminalBlock_Phoenix_MPT-0,5-4-2.54_1x04_P2.54mm_Horizontal, F.Cu at (99.1, 107.2)
- added R52: 10k, Resistor_SMD:R_0603_1608Metric, F.Cu at (126.5, 42.0)
- added R53: 210, Resistor_SMD:R_0603_1608Metric, F.Cu at (123.5, 42.0)
- added R54: 400, Resistor_SMD:R_0603_1608Metric, F.Cu at (120.5, 42.0)
- added R61: 210, Resistor_SMD:R_0603_1608Metric, F.Cu at (117.5, 42.0)
- added TP1: GND, TestPoint:TestPoint_Loop_D2.50mm_Drill1.85mm, F.Cu at (135.5, 113.5)
- added TP2: VCC, TestPoint:TestPoint_Loop_D2.50mm_Drill1.85mm, F.Cu at (129.0, 111.5)
- added TP3: 3.3V, TestPoint:TestPoint_Loop_D2.50mm_Drill1.85mm, F.Cu at (129.0, 93.5)
- added TP4: 5V, TestPoint:TestPoint_Loop_D2.50mm_Drill1.85mm, F.Cu at (125.0, 97.5)
- added kibuzzard-6AC244AE: G***, kibuzzard-6AC244AE, F.Cu at (104.0, 111.0)
- added kibuzzard-6AC244BE: G***, kibuzzard-6AC244BE, F.Cu at (104.0, 97.0)
- D10, D6, D7, D8: footprint Diode_SMD:D_SOD-123 -> Diode_SMD:D_0603_1608Metric
- J8: value RJ45_Wuerth_7499010211A -> VCC; footprint Connector_RJ:RJ45_Wuerth_7499010211A_Horizontal -> TerminalBlock_Phoenix:TerminalBlock_Phoenix_MPT-0,5-4-2.54_1x04_P2.54mm_Horizontal
- R1, R10, R11, R12, R13, R14, R15, R16, R17, R18, R19, R2, R3, R32, R33, R34, R35, R36, R37, R38, R39, R4, R40, R45, R46, R47, R48, R49, R5, R50, R51, R55, R56, R57, R6, R63, R7, R77, R8, R9: footprint Resistor_SMD:R_0805_2012Metric -> Resistor_SMD:R_0603_1608Metric
- moved H3 130.7 mm to (63.0, 70.2)
- moved H2 119.1 mm to (63.0, 64.5)
- moved H1 85.0 mm to (173.0, 43.0)
- moved M1 79.4 mm to (77.2, 72.7), turned to 0 degrees
- moved D3 72.9 mm to (108.0, 106.5), turned to 180 degrees
- moved R4 70.6 mm to (107.5, 103.5), turned to 0 degrees
- moved J2 70.0 mm to (105.8, 79.5), turned to -90 degrees
- moved J6 68.8 mm to (136.3, 68.8)
- moved C16 63.2 mm to (116.5, 111.0), turned to -90 degrees
- moved Q1 60.1 mm to (109.0, 96.0), turned to 90 degrees
- moved H4 55.7 mm to (63.0, 76.0)
- moved F1 54.9 mm to (118.7, 85.0)
- moved J4 47.6 mm to (171.9, 100.8), turned to 90 degrees
- moved J9 45.4 mm to (172.0, 86.8), turned to 90 degrees
- moved J5 43.8 mm to (167.6, 49.0), turned to -90 degrees
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Connections:
- J8 pad 1: /ETH_TX_B_P -> VCC
- J8 pad 2: /ETH_TX_B_N -> VCC
- J8 pad 3: /ETH_RX_C_P -> VCC
- J8 pad 4: Net-(J8-CTD) -> VCC
- U1 pad 19: unconnected-(U1-IO11-Pad19) -> Pin1
- U1 pad 20: unconnected-(U1-IO12-Pad20) -> Pin2
- U1 pad 21: unconnected-(U1-IO13-Pad21) -> Pin3
- U1 pad 22: unconnected-(U1-IO14-Pad22) -> Pin4
- U1 pad 24: unconnected-(U1-IO47-Pad24) -> Pin5
- U1 pad 25: unconnected-(U1-IO48-Pad25) -> Pin6
- U1 pad 31: ETH_CS -> Pin7
Routing:
- net MISO: track 110.9 -> 0.00 mm, vias 4 -> 0
- net MOSI: track 110.8 -> 0.00 mm, vias 4 -> 0
- net SCLK: track 103.3 -> 0.00 mm, vias 4 -> 0
- net CS_ADC: track 89.8 -> 0.00 mm, vias 2 -> 0
- net +5V: track 87.7 -> 31.8 mm, vias 3 -> 0
- net ACT_LED: track 53.7 -> 0.00 mm, vias 2 -> 0
- net RST: track 81.5 -> 30.7 mm, vias 3 -> 2
- net LINK_LED: track 46.6 -> 0.00 mm, vias 2 -> 0
- net +3.3VA: track 32.3 -> 0.00 mm, vias 6 -> 0
- net ETH_CS: track 31.5 -> 0.00 mm, vias 2 -> 0
- net CURR1: track 27.7 -> 58.0 mm
- net Net-(U1-IO0): track 25.8 -> 0.00 mm
- net /shield: track 24.6 -> 0.00 mm
- net NTC1: track 34.6 -> 15.2 mm, vias 4 -> 0
- net +3.3V: track 98.5 -> 79.2 mm, vias 158 -> 72
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- added copper zone on B.Cu, net +3.3V
- added copper zone on In2.Cu, net GND
- removed copper zone on In2.Cu, net +3.3V
- removed copper zone on In2.Cu, net +3.3VA
- removed copper zone on B.Cu, net GND
- removed copper zone on F.Cu, net IO1
- removed copper zone on F.Cu, net IO2
- removed copper zone on F.Cu, net IO3
- removed copper zone on F.Cu, net IO4
- removed copper zone on B.Cu, net Net-(D4-A1)
- removed copper zone on B.Cu, net Net-(J2-Pin_2)
Other:
- board size 100 x 80 mm -> 81 x 85 mm
- board text removed: "Track width: (etehrnet) 0.5 oz inner:0.3051 1oz inner: 0,2722mm spacing: 0.5mm"

Commit message: I cant do this anymore
Signed-off-by: Peter Schmidt <hackepetersilie@gmx.de>
Parts:
- moved R32 42.5 mm to (158.2, 63.0), turned to 0 degrees
- moved M1 41.6 mm to (118.7, 69.2)
- moved R33 41.5 mm to (158.2, 61.5), turned to 180 degrees
- moved R34 40.5 mm to (158.2, 60.0), turned to 0 degrees
- moved R35 39.6 mm to (158.2, 58.5), turned to 180 degrees
- moved D6 38.9 mm to (155.2, 63.0), turned to 180 degrees
- moved R36 38.9 mm to (158.2, 57.0), turned to 0 degrees
- moved R37 38.2 mm to (158.2, 55.5), turned to 180 degrees
- moved R45 37.8 mm to (155.2, 61.5), turned to 180 degrees
- moved R38 37.6 mm to (158.2, 54.0), turned to 0 degrees
- moved R39 37.2 mm to (158.2, 52.5), turned to 180 degrees
- moved D7 36.7 mm to (155.2, 60.0), turned to 180 degrees
- moved R46 35.8 mm to (155.2, 58.5), turned to 180 degrees
- moved D8 34.9 mm to (155.2, 57.0), turned to 180 degrees
- moved R47 34.2 mm to (155.2, 55.5), turned to 180 degrees
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Routing:
- net +3.3V: track 79.2 -> 199.8 mm, vias 72 -> 74
- net IN1.1: track 2.06 -> 97.3 mm, vias 1 -> 3
- net IN1.2: track 0.92 -> 92.2 mm, vias 1 -> 3
- net IN2.2: track 2.06 -> 88.5 mm, vias 1 -> 2
- net +5V: track 31.8 -> 99.3 mm, vias 0 -> 1
- net OUT5: track 0.00 -> 62.6 mm, vias 0 -> 2
- net IN2.1: track 0.92 -> 63.1 mm, vias 1 -> 2
- net OUT6: track 0.00 -> 61.3 mm, vias 0 -> 3
- net OUT7: track 0.00 -> 58.2 mm, vias 0 -> 3
- net OUT8: track 0.00 -> 52.9 mm, vias 0 -> 3
- net MISO: track 0.00 -> 51.2 mm, vias 0 -> 2
- net MOSI: track 0.00 -> 51.1 mm, vias 0 -> 2
- net IO1: track 12.0 -> 62.5 mm, vias 0 -> 1
- net IO2: track 11.2 -> 60.0 mm, vias 0 -> 1
- net IO3: track 12.6 -> 61.1 mm, vias 0 -> 1
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
Commit message: DONE!!!
Parts:
- removed M1: Fan_4pin, Connector:FanPinHeader_1x04_P2.54mm_Vertical
- removed kibuzzard-6AC244AE: G***, kibuzzard-6AC244AE
- removed kibuzzard-6AC244BE: G***, kibuzzard-6AC244BE
- added C19: 100nF, Capacitor_SMD:C_0603_1608Metric, F.Cu at (120.0, 55.0)
- added C20: 22uF, Capacitor_SMD:C_0603_1608Metric, F.Cu at (117.5, 55.0)
- added kibuzzard-6ACBD168: G***, kibuzzard-6ACBD168, F.Cu at (167.5, 116.5)
- added kibuzzard-6ACBD1B3: G***, kibuzzard-6ACBD1B3, F.Cu at (167.5, 104.0)
- added kibuzzard-6ACBD341: G***, kibuzzard-6ACBD341, F.Cu at (112.5, 99.0)
- added kibuzzard-6ACBD34D: G***, kibuzzard-6ACBD34D, F.Cu at (112.5, 110.5)
- added kibuzzard-6ACBD3AA: G***, kibuzzard-6ACBD3AA, F.Cu at (104.5, 112.2)
- added kibuzzard-6ACBD3B0: G***, kibuzzard-6ACBD3B0, F.Cu at (104.5, 114.8)
- added kibuzzard-6ACBD3CF: G***, kibuzzard-6ACBD3CF, F.Cu at (104.5, 117.2)
- added kibuzzard-6ACBD3D5: G***, kibuzzard-6ACBD3D5, F.Cu at (104.5, 119.8)
- added kibuzzard-6ACBD409: G***, kibuzzard-6ACBD409, F.Cu at (104.2, 129.2)
- added kibuzzard-6ACBD410: G***, kibuzzard-6ACBD410, F.Cu at (104.2, 126.8)
- added kibuzzard-6ACBD41A: G***, kibuzzard-6ACBD41A, F.Cu at (104.2, 124.2)
- added kibuzzard-6ACBD423: G***, kibuzzard-6ACBD423, F.Cu at (104.2, 131.8)
- added kibuzzard-6ACBD433: G***, kibuzzard-6ACBD433, F.Cu at (167.5, 128.0)
- added kibuzzard-6ACBD473: G***, kibuzzard-6ACBD473, F.Cu at (155.8, 61.2)
- added kibuzzard-6ACBD50A: G***, kibuzzard-6ACBD50A, F.Cu at (100.2, 69.0)
- added kibuzzard-6ACBD573: G***, kibuzzard-6ACBD573, F.Cu at (170.0, 70.2)
- added kibuzzard-6ACBD5D3: G***, kibuzzard-6ACBD5D3, F.Cu at (161.5, 73.5)
- added kibuzzard-6ACBD5E0: G***, kibuzzard-6ACBD5E0, F.Cu at (153.2, 73.5)
- moved H4 126.8 mm to (173.0, 139.0)
- moved J9 77.4 mm to (98.9, 112.2), turned to -90 degrees
- moved H3 77.1 mm to (98.0, 139.0)
- moved J4 76.6 mm to (98.9, 124.2), turned to -90 degrees
- moved J8 74.6 mm to (172.2, 108.0), turned to 90 degrees
- moved J7 74.2 mm to (172.2, 120.0), turned to 90 degrees
- moved R18 72.4 mm to (109.0, 121.5), turned to 0 degrees
- moved D12 71.4 mm to (174.0, 91.0), turned to -90 degrees
- moved R19 70.6 mm to (109.0, 120.0), turned to 180 degrees
- moved R53 69.3 mm to (172.5, 91.0), turned to -90 degrees
- moved R16 68.9 mm to (109.0, 118.5), turned to 0 degrees
- moved D13 68.6 mm to (174.0, 83.0), turned to -90 degrees
- moved R17 67.3 mm to (109.0, 117.0), turned to 180 degrees
- moved D11 66.5 mm to (174.0, 87.0), turned to -90 degrees
- moved R54 66.2 mm to (172.5, 83.0), turned to -90 degrees
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Connections:
- U1 pad 10: IN7 -> SCL
- U1 pad 11: IN8 -> SDA
- U1 pad 12: OUT8 -> LED1
- U1 pad 15: IN2.1 -> IN5
- U1 pad 16: Net-(M1-PWM) -> unconnected-(U1-IO46-Pad16)
- U1 pad 17: SDA -> IN7
- U1 pad 18: SCL -> IN8
- U1 pad 19: Pin1 -> OUT5
- U1 pad 20: Pin2 -> OUT6
- U1 pad 21: Pin3 -> OUT7
- U1 pad 22: Pin4 -> OUT8
- U1 pad 23: LED1 -> IN1.2
- U1 pad 24: Pin5 -> IN1.1
- U1 pad 25: Pin6 -> IN6
- U1 pad 26: Net-(M1-Tacho) -> unconnected-(U1-IO45-Pad26)
- U1 pad 31: Pin7 -> IN2.2
- U1 pad 32: SCLK -> IN2.1
- U1 pad 33: MOSI -> CS_ADC
- U1 pad 34: MISO -> SCLK
- U1 pad 35: CS_ADC -> MISO
- U1 pad 38: IN1.2 -> MOSI
- U1 pad 39: IN1.1 -> Pin7
- U1 pad 4: IN2.2 -> Pin6
- U1 pad 5: OUT5 -> Pin5
- U1 pad 6: OUT6 -> Pin4
- U1 pad 7: OUT7 -> Pin3
- U1 pad 8: IN5 -> Pin2
- U1 pad 9: IN6 -> Pin1
Routing:
- net +3.3V: track 199.8 -> 58.4 mm, vias 74 -> 239
- net VCC: track 157.5 -> 210.1 mm, vias 70 -> 14
- net MOSI: track 51.1 -> 101.5 mm, vias 2 -> 1
- net SCLK: track 48.0 -> 93.1 mm
- net MISO: track 51.2 -> 94.8 mm, vias 2 -> 1
- net Pin1: track 0.00 -> 40.2 mm
- net Pin2: track 0.00 -> 38.1 mm
- net Pin3: track 0.00 -> 37.2 mm
- net Pin4: track 0.00 -> 35.8 mm
- net Pin5: track 0.00 -> 34.5 mm
- net Pin7: track 0.00 -> 33.4 mm
- net Pin6: track 0.00 -> 33.3 mm
- net D+: track 0.00 -> 31.2 mm
- net D-: track 0.00 -> 31.2 mm
- net CS_ADC: track 36.9 -> 67.2 mm, vias 0 -> 2
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- added copper zone on In2.Cu, net +3.3V
- added copper zone on F.Cu, net IO1
- added copper zone on F.Cu, net IO2
- added copper zone on F.Cu, net IO3
- added copper zone on F.Cu, net IO4
- removed copper zone on In2.Cu, net GND
- removed copper zone on F.Cu, net Net-(D22-A)
- removed copper zone on F.Cu, net Net-(D4-A1)
- removed copper zone on F.Cu, net Net-(J2-Pin_2)
Other:
- board size 81 x 85 mm -> 81 x 90.2 mm
