File: MildlyOverkill.kicad_pcb (KiCad board)
At the start: 4 copper layers, 81 x 90.2 mm, 130 parts, among them J1 USB_C_Receptacle_USB2.0_16P, J10 Conn_01x07_Pin, J11 Conn_01x08_Pin, J2 Screw_Terminal_01x02, J3 Motors, J4 IO, J5 Conn_01x04_Pin, J6 Conn_01x04_MountingPin, J7 GND, J8 VCC, J9 Analog, Q1 Q_PMOS_GDS, U1 ESP32-S3-WROOM-1, U2 MCP3208, U3 LD1117S33TR_SOT223, U4 TPS4H160AQPWPRQ1, U5 USBLC6-2P6, U6 TPS62932, U8 DRV8874PWPR, U9 DRV8874PWPR

Commit message: Done for now
Parts:
- added kibuzzard-6ACBE024: G***, kibuzzard-6ACBE024, F.Cu at (119.0, 71.2)
Routing:
- net +3.3V: track 58.4 -> 82.7 mm, vias 239 -> 212
- added copper zone on B.Cu, net GND
- removed copper zone on B.Cu, net +3.3V

Commit message: Added todo and a lot of more or less minor changes
Parts:
- C11: footprint Capacitor_SMD:C_0603_1608Metric -> Capacitor_SMD:C_0805_2012Metric
- D10, D6, D7, D8: footprint Diode_SMD:D_0603_1608Metric -> Diode_SMD:D_SOD-323
- D22: value D_Schottky -> B5819W
- D5: value D_Schottky -> B5819W; footprint Diode_SMD:D_SOD-123 -> Diode_SMD:D_SOD-323
- FB1: value FerriteBead -> BLM21PG221SN1
- Q1: value Q_PMOS_GDS -> AOD4185
- R11, R8: value 3300 -> 2.37k
- R4: value 100 -> 100k
- moved D10 0.86 mm to (129.8, 82.5)
- moved D6 0.86 mm to (122.8, 82.5)
- moved D8 0.86 mm to (126.2, 82.5)
- moved D7 0.72 mm to (145.0, 77.5)
- moved C11 0.35 mm to (148.8, 89.8)
Connections:
- R63 pad 1: GND -> +3.3V
Routing:
- net +3.3V: track 82.7 -> 83.9 mm, vias 212 -> 213
- net Net-(D6-K): track 4.20 -> 5.22 mm
- net Net-(D10-K): track 4.20 -> 5.19 mm
- net Net-(D8-K): track 4.19 -> 5.14 mm
- net Net-(D5-A): track 2.29 -> 2.89 mm
- net +5V: track 87.2 -> 87.8 mm
- net Net-(D7-K): track 4.20 -> 4.77 mm
- net GND: vias 72 -> 73

Commit message: Did some stuff on the todo list TL;DR:The piece of meat did what the thinking sand said and now it can sleep in peace. The end.
Parts:
- added C21: 10uF 50V, Capacitor_SMD:C_1210_3225Metric, F.Cu at (160.2, 115.8)
- added C22: 10uF 50V, Capacitor_SMD:C_1210_3225Metric, F.Cu at (164.0, 139.2)
- added C23: 0.1uF 50V, Capacitor_SMD:C_0603_1608Metric, F.Cu at (112.6, 138.4)
- added C24: 10uF 50V, Capacitor_SMD:C_1210_3225Metric, F.Cu at (112.6, 135.4)
- added C25: 2.2uF, Capacitor_SMD:C_1206_3216Metric, F.Cu at (109.9, 92.7)
- added R20: 4.7k, Resistor_SMD:R_0805_2012Metric_Pad1.20x1.40mm_HandSolder, F.Cu at (118.0, 75.5)
- added R21: 4.7k, Resistor_SMD:R_0805_2012Metric_Pad1.20x1.40mm_HandSolder, F.Cu at (115.0, 75.5)
- C1: value 100nF -> 1uF 10V
- C11: value 47uF -> 47uF 10V X5R
- C13: value 100nF -> 100nF 50V
- C14: value 10uF -> 10uF 50V
- C15, C7, C8, C9: value 0.1uF -> 0.1uF 50V
- C16: value 1000uF -> 1000uF 35V
- C17: value 10uF -> 10uF 10V X5R
- C18, C6: value 0.022uF -> 0.022uF 50V
- C20: value 22uF -> 22uF 10V X5R
- D10, D6, D7, D8: value 3v -> BZT52C3V0S
- D3: footprint Diode_SMD:D_0805_2012Metric -> Diode_SMD:D_SOD-123
- D4: value SMAJ33A -> SMAJ24CA
- D5: footprint Diode_SMD:D_SOD-323 -> Diode_SMD:D_SOD-123
- F1: value Fuse -> 10A
- R1: value 5,1K -> 10k
- R10, R9: value 660 -> 665
- R3, R5: value 5,1K -> 5.1k
- R32, R34, R36, R38: value 3k -> 3.01k
- R33, R35, R37, R39: value 6k -> 6.04k
- R54: value 400 -> 402
- R77: value R -> 10k 1%
- TH1: value Thermistor_NTC -> NCP18XH103F03RB
- U3: value LD1117S33TR_SOT223 -> AP7361C-33E
- moved C4 13.2 mm to (154.8, 94.0)
- moved U3 4.76 mm to (156.8, 88.8)
Connections:
- U3 pad 1: GND -> +5V
- U3 pad 2: +3.3V -> GND
- U3 pad 3: +5V -> +3.3V
Routing:
- net VCC: track 210.1 -> 289.4 mm, vias 14 -> 25
- net +3.3V: track 83.9 -> 101.8 mm, vias 213 -> 27
- net SCL: track 15.6 -> 23.5 mm, vias 0 -> 2
- net SDA: track 17.7 -> 22.9 mm, vias 0 -> 2
- net ST: track 26.3 -> 29.9 mm
- net CURR2: track 24.8 -> 21.8 mm, vias 2 -> 0
- net GND: track 29.0 -> 27.0 mm, vias 73 -> 83
- net Net-(D5-A): track 2.89 -> 4.82 mm
- net CURR1: track 34.0 -> 35.7 mm
- net RX: track 8.18 -> 7.54 mm
- net +5V: track 87.8 -> 87.2 mm
- removed copper zone on F.Cu, net +3.3V
