File: H-Bridge.kicad_sch (KiCad schematic)
At the start: 7 parts, among them U8 DRV8874PWPR

Commit message: idk where to begin...
Parts:
- R8, R9: footprint Resistor_SMD:R_0805_2012Metric -> Resistor_SMD:R_0603_1608Metric
Changed lines of the file:
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@@
 			)
 		)
-		(property "Footprint" "Resistor_SMD:R_0805_2012Metric"
+		(property "Footprint" "Resistor_SMD:R_0603_1608Metric"
 			(at 55.372 119.38 90)
 			(hide yes)
@@
 			)
 		)
-		(property "Footprint" "Resistor_SMD:R_0805_2012Metric"
+		(property "Footprint" "Resistor_SMD:R_0603_1608Metric"
 			(at 52.832 88.9 90)
 			(hide yes)

Commit message: Added todo and a lot of more or less minor changes
Parts:
- R8: value 3300 -> 2.37k
Changed lines of the file:
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@@
 			)
 		)
-		(property "Value" "3300"
+		(property "Value" "2.37k"
 			(at 59.69 120.6499 0)
 			(show_name no)
