File: H-Bridge.kicad_sch (KiCad schematic)
At the start: 7 parts, among them U8 DRV8874PWPR

Commit message: BOM cleanup: values, MPNs and voltage ratings from todo.md
Values/fields only, no footprint or net changes (netlist diff is empty).

Co-Authored-By: Claude Sonnet 5.5 <noreply@anthropic.com> (obviously)
Parts:
- C6: value 0.022uF -> 0.022uF 50V
- C7, C8: value 0.1uF -> 0.1uF 50V
- R9: value 660 -> 665
Changed lines of the file:
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@@
 			)
 		)
-		(property "Value" "0.1uF"
+		(property "Value" "0.1uF 50V"
 			(at 43.688 76.454 90)
 			(show_name no)
@@
 			)
 		)
-		(property "Value" "0.022uF"
+		(property "Value" "0.022uF 50V"
 			(at 116.84 106.6799 0)
 			(show_name no)
@@
 			)
 		)
-		(property "Value" "660"
+		(property "Value" "665"
 			(at 57.15 90.1699 0)
 			(show_name no)
@@
 			)
 		)
-		(property "Value" "0.1uF"
+		(property "Value" "0.1uF 50V"
 			(at 65.786 85.598 90)
 			(show_name no)
