File: H-Bridge.kicad_sch (KiCad schematic)
At the start: 7 parts, among them U8 DRV8874PWPR

Commit message: Did some stuff on the todo list TL;DR:The piece of meat did what the thinking sand said and now it can sleep in peace. The end.
Parts:
- added C21: 10uF 50V, Capacitor_SMD:C_1210_3225Metric, symbol Device:C
Connections:
- net GND: now also C21.2
- net VIN: now also C21.1
Other:
- moved on the sheet: C8
