File: weakIO.kicad_sch (KiCad schematic)
At the start: 25 parts, among them U4 TPS4H160AQPWPRQ1

Commit message: BOM cleanup: values, MPNs and voltage ratings from todo.md
Values/fields only, no footprint or net changes (netlist diff is empty).

Co-Authored-By: Claude Sonnet 5.5 <noreply@anthropic.com> (obviously)
Parts:
- D10, D6, D7, D8: value 3v -> BZT52C3V0S
- R32, R34, R36, R38: value 3k -> 3.01k
- R33, R35, R37, R39: value 6k -> 6.04k
Changed lines of the file:
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@@
 			)
 		)
-		(property "Value" "3k"
+		(property "Value" "3.01k"
 			(at 162.56 52.0699 0)
 			(show_name no)
@@
 			)
 		)
-		(property "Value" "6k"
+		(property "Value" "6.04k"
 			(at 171.45 73.6599 0)
 			(show_name no)
@@
 			)
 		)
-		(property "Value" "3k"
+		(property "Value" "3.01k"
 			(at 162.56 146.0499 0)
 			(show_name no)
@@
 			)
 		)
-		(property "Value" "3k"
+		(property "Value" "3.01k"
 			(at 162.56 115.5699 0)
 			(show_name no)
@@
 			)
 		)
-		(property "Value" "6k"
+		(property "Value" "6.04k"
 			(at 171.45 105.4099 0)
 			(show_name no)
@@
 			)
 		)
-		(property "Value" "3v"
+		(property "Value" "BZT52C3V0S"
 			(at 171.45 83.8199 90)
 			(show_name no)
@@
 			)
 		)
-		(property "Value" "3v"
+		(property "Value" "BZT52C3V0S"
 			(at 171.45 52.0699 90)
 			(show_name no)
@@
 			)
 		)
-		(property "Value" "6k"
+		(property "Value" "6.04k"
 			(at 171.45 41.9099 0)
 			(show_name no)
@@
 			)
 		)
-		(property "Value" "3v"
+		(property "Value" "BZT52C3V0S"
 			(at 171.45 146.0499 90)
 			(show_name no)
@@
 			)
 		)
-		(property "Value" "3k"
+		(property "Value" "3.01k"
 			(at 162.56 83.8199 0)
 			(show_name no)
@@
 			)
 		)
-		(property "Value" "3v"
+		(property "Value" "BZT52C3V0S"
 			(at 171.45 115.5699 90)
 			(show_name no)
@@
 			)
 		)
-		(property "Value" "6k"
+		(property "Value" "6.04k"
 			(at 171.45 135.8899 0)
 			(show_name no)
