File: weakIO.kicad_sch (KiCad schematic)
At the start: 25 parts, among them U4 TPS4H160AQPWPRQ1

Commit message: Did some stuff on the todo list TL;DR:The piece of meat did what the thinking sand said and now it can sleep in peace. The end.
Parts:
- added C23: 0.1uF 50V, Capacitor_SMD:C_0603_1608Metric, symbol Device:C
- added C24: 10uF 50V, Capacitor_SMD:C_1210_3225Metric, symbol Device:C
Connections:
- net EXP: now also C23.1, C24.2
- net VS: now also C23.2, C24.1
